File: Системи автоматизованого проектування електронних пристроїв і сигналів (Кн+)/Lab1/Lab1/_autosave-Lab1.kicad_sch (KiCad schematic)
At the start: 1 part, among them Q1 2SA1015

Commit message: update
Parts:
- added U1: AD40xxBCPZ, Package_CSP:LFCSP-WD-10-1EP_3x3mm_P0.5mm_EP1.64x2.38mm, symbol Analog_ADC:AD40xxBCPZ
Connections:
- net at Q1.1 (E), Q1.2 (C): now also U1.1 (REF)
Changed lines of the file:
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@@
 	(generator_version "8.0")
 	(paper "A4")
+	(junction
+		(at 96.52 76.2)
+		(diameter 0)
+		(color 0 0 0 0)
+	)
 	(wire
 		(pts
 			(xy 96.52 76.2) (xy 80.01 76.2)
+		)
+		(stroke
+			(width 0)
+			(type default)
+		)
+	)
+	(wire
+		(pts
+			(xy 101.6 76.2) (xy 101.6 80.01)
 		)
 		(stroke
@@
 	(wire
 		(pts
+			(xy 96.52 76.2) (xy 101.6 76.2)
+		)
+		(stroke
+			(width 0)
+			(type default)
+		)
+	)
+	(wire
+		(pts
 			(xy 96.52 60.96) (xy 96.52 76.2)
 		)
@@
 		)
 	)
+	(symbol
+		(lib_id "Analog_ADC:AD40xxBCPZ")
+		(at 104.14 90.17 0)
+		(unit 1)
+		(exclude_from_sim no)
+		(in_bom yes)
+		(on_board yes)
+		(dnp no)
+		(fields_autoplaced yes)
+		(property "Reference" "U1"
+			(at 83.82 81.3114 0)
+			(effects
+				(font
+					(size 1.27 1.27)
+				)
+			)
+		)
+		(property "Value" "AD40xxBCPZ"
+			(at 83.82 83.8514 0)
+			(effects
+				(font
+					(size 1.27 1.27)
+				)
+			)
+		)
+		(property "Footprint" "Package_CSP:LFCSP-WD-10-1EP_3x3mm_P0.5mm_EP1.64x2.38mm"
+			(at 104.14 110.49 0)
+			(effects
+				(font
+					(size 1.27 1.27)
+				)
+				(hide yes)
+			)
+		)
+		(property "Datasheet" "https://www.analog.com/media/en/technical-documentation/data-sheets/ad4003-4007-4011.pdf"
+			(at 104.14 113.03 0)
+			(effects
+				(font
+					(size 1.27 1.27)
+				)
+				(hide yes)
+			)
+		)
+		(property "Description" "18-Bit, 2 MSPS/1 MSPS/500 kSPS, Differential SAR ADCs, 2.4V to 5.1V reference, 1.8V supply, 1.71 to 5.5V logic IO, 3x3mm LFCSP-10"
+			(at 104.14 90.17 0)
+			(effects
+				(font
+					(size 1.27 1.27)
+				)
+				(hide yes)
+			)
+		)
+		(pin "5"
+		)
+		(pin "2"
+		)
+		(pin "1"
+		)
+		(pin "7"
+		)
+		(pin "3"
+		)
+		(pin "10"
+		)
+		(pin "11"
+		)
+		(pin "6"
+		)
+		(pin "9"
+		)
+		(pin "8"
+		)
+		(pin "4"
+		)
+		(instances
+			(project ""
+				(path "/d90ba17d-fee1-41fe-8a12-45c540d367c6"
+					(reference "U1")
+					(unit 1)
+				)
+			)
+		)
+	)
